Commit message: changed pkg name in launch files

File: diffdrive_arduino/description/ros2_control/diffbot.ros2_control.xacro (robot description, xacro)
@@ -4,5 +4,13 @@
     <ros2_control name="${name}" type="system">
       <hardware>
-        <plugin>diffdrive_arduino/DiffDriveArduinoHardware</plugin>
+      <plugin>diffdrive_arduino/DiffDriveArduinoHardware</plugin>
+        <param name="left_wheel_name">BL_joint</param>
+        <param name="right_wheel_name">BR_joint</param>
+        <param name="loop_rate">30</param>
+        <param name="device">/dev/ttyUSB0</param>
+        <param name="baud_rate">57600</param>
+        <param name="timeout_ms">1000</param>
+        <param name="enc_counts_per_rev">2952</param>
+        <!-- <plugin>diffdrive_arduino/DiffDriveArduinoHardware</plugin>
         <param name="left_wheel_name">left_wheel_joint</param>
         <param name="right_wheel_name">right_wheel_joint</param>
@@ -11,5 +19,5 @@
         <param name="baud_rate">57600</param>
         <param name="timeout_ms">1000</param>
-        <param name="enc_counts_per_rev">3436</param>
+        <param name="enc_counts_per_rev">3436</param> -->
         <param name="pid_p">20</param>
         <param name="pid_d">12</param>
@@ -17,10 +25,10 @@
         <param name="pid_o">50</param>
       </hardware>
-      <joint name="${prefix}left_wheel_joint">
+      <joint name="${prefix}BL_joint">
         <command_interface name="velocity"/>
         <state_interface name="position"/>
         <state_interface name="velocity"/>
       </joint>
-      <joint name="${prefix}right_wheel_joint">
+      <joint name="${prefix}BR_joint">
         <command_interface name="velocity"/>
         <state_interface name="position"/>
