Commit message: removed .git folder

File: cvr_bot_description/urdf/cvr_bot_sim.xacro (robot description, xacro)
@@ -44,5 +44,5 @@
     <origin xyz="0 0 0" rpy="0 0 0"/>
     <geometry>
-      <mesh filename="file://$(find cvr_bot_description)/meshes/base_link.dae" scale="0.001 0.001 0.001"/>
+      <mesh filename="package://cvr_bot_description/meshes/base_link.dae" scale="0.001 0.001 0.001"/>
     </geometry>
     <material name="blue"/>
@@ -51,5 +51,5 @@
     <origin xyz="0 0 0.115" rpy="0 0 0"/>
     <geometry>
-      <!-- <mesh filename="file://$(find cvr_bot_description)/meshes/base_link.dae" scale="0.001 0.001 0.001"/> -->
+      <!-- <mesh filename="package://cvr_bot_description/meshes/base_link.dae" scale="0.001 0.001 0.001"/> -->
       <box size="0.29 0.29 0.23"/>
     </geometry>
@@ -69,5 +69,5 @@
     <origin xyz="0.094914 0.152452 -0.064084" rpy="0 0 0"/>
     <geometry>
-      <mesh filename="file://$(find cvr_bot_description)/meshes/br_wheel_2.dae" scale="0.001 0.001 0.001"/>
+      <mesh filename="package://cvr_bot_description/meshes/br_wheel_2.dae" scale="0.001 0.001 0.001"/>
     </geometry>
     <material name="silver"/>
@@ -76,5 +76,5 @@
     <!-- <origin xyz="0.094914 0.152452 -0.064084" rpy="0 0 0"/> -->
     <geometry>
-      <!-- <mesh filename="file://$(find cvr_bot_description)/meshes/br_wheel_2.dae" scale="0.001 0.001 0.001"/> -->
+      <!-- <mesh filename="package://cvr_bot_description/meshes/br_wheel_2.dae" scale="0.001 0.001 0.001"/> -->
       <sphere radius="${wheel_radius}"/>
     </geometry>
@@ -91,5 +91,5 @@
     <origin xyz="-0.095849 0.151214 -0.062584" rpy="0 0 0"/>
     <geometry>
-      <mesh filename="file://$(find cvr_bot_description)/meshes/fr_wheel.dae" scale="0.001 0.001 0.001"/>
+      <mesh filename="package://cvr_bot_description/meshes/fr_wheel.dae" scale="0.001 0.001 0.001"/>
     </geometry>
     <material name="silver"/>
@@ -98,5 +98,5 @@
     <!-- <origin xyz="-0.095849 0.151214 -0.062584" rpy="0 0 0"/> -->
     <geometry>
-      <!-- <mesh filename="file://$(find cvr_bot_description)/meshes/fr_wheel.dae" scale="0.001 0.001 0.001"/> -->
+      <!-- <mesh filename="package://cvr_bot_description/meshes/fr_wheel.dae" scale="0.001 0.001 0.001"/> -->
       <sphere radius="${wheel_radius}"/>
     </geometry>
@@ -113,5 +113,5 @@
     <origin xyz="-0.095849 -0.162786 -0.062584" rpy="0 0 0"/>
     <geometry>
-      <mesh filename="file://$(find cvr_bot_description)/meshes/fl_wheel.dae" scale="0.001 0.001 0.001"/>
+      <mesh filename="package://cvr_bot_description/meshes/fl_wheel.dae" scale="0.001 0.001 0.001"/>
     </geometry>
     <material name="silver"/>
@@ -120,5 +120,5 @@
     <!-- <origin xyz="-0.095849 -0.162786 -0.062584" rpy="0 0 0"/> -->
     <geometry>
-      <!-- <mesh filename="file://$(find cvr_bot_description)/meshes/fl_wheel.dae" scale="0.001 0.001 0.001"/> -->
+      <!-- <mesh filename="package://cvr_bot_description/meshes/fl_wheel.dae" scale="0.001 0.001 0.001"/> -->
       <sphere radius="${wheel_radius}"/>
     </geometry>
@@ -135,5 +135,5 @@
     <origin xyz="0.096151 -0.162786 -0.062584" rpy="0 0 0"/>
     <geometry>
-      <mesh filename="file://$(find cvr_bot_description)/meshes/bl_wheel.dae" scale="0.001 0.001 0.001"/>
+      <mesh filename="package://cvr_bot_description/meshes/bl_wheel.dae" scale="0.001 0.001 0.001"/>
     </geometry>
     <material name="silver"/>
@@ -142,5 +142,5 @@
     <!-- <origin xyz="0.096151 -0.162786 -0.062584" rpy="0 0 0"/> -->
     <geometry>
-      <!-- <mesh filename="file://$(find cvr_bot_description)/meshes/bl_wheel.dae" scale="0.001 0.001 0.001"/> -->
+      <!-- <mesh filename="package://cvr_bot_description/meshes/bl_wheel.dae" scale="0.001 0.001 0.001"/> -->
       <sphere radius="${wheel_radius}"/>
     </geometry>
@@ -215,5 +215,5 @@
     <origin xyz="0 0 0" rpy="0 0 0" />
     <geometry>
-      <mesh filename="file://$(find cvr_bot_description)/meshes/laser_link.STL" />
+      <mesh filename="package://cvr_bot_description/meshes/laser_link.STL" />
     </geometry>
     <material name="black"/>
@@ -222,5 +222,5 @@
     <origin xyz="0 0 0" rpy="0 0 0" />
     <geometry>
-      <mesh filename="file://$(find cvr_bot_description)/meshes/laser_link.STL" />
+      <mesh filename="package://cvr_bot_description/meshes/laser_link.STL" />
     </geometry>
   </collision>

File: cvr_bot_description/urdf/ros2_control.xacro (robot description, xacro)
@@ -7,4 +7,6 @@
                 <param name="left_wheel_name">BL_joint</param>
                 <param name="right_wheel_name">BR_joint</param>
+                <param name="left1_wheel_name">FL_joint</param>
+                <param name="right1_wheel_name">FR_joint</param>
                 <param name="loop_rate">30</param>
                 <param name="device">/dev/ttyUSB0</param>
@@ -14,4 +16,43 @@
             </hardware>
             <joint name="FL_joint">
+                <command_interface name="velocity">
+                    <param name="min">-10</param>
+                    <param name="max">10</param>
+                </command_interface>
+                <state_interface name="position"/>
+                <state_interface name="velocity"/>
+            </joint>
+            <joint name="FR_joint">
+                <command_interface name="velocity">
+                    <param name="min">-10</param>
+                    <param name="max">10</param>
+                </command_interface>
+                <state_interface name="position"/>
+                <state_interface name="velocity"/>
+            </joint>
+            <joint name="BL_joint">
+                <command_interface name="velocity">
+                    <param name="min">-10</param>
+                    <param name="max">10</param>
+                </command_interface>
+                <state_interface name="position"/>
+                <state_interface name="velocity"/>
+            </joint>
+            <joint name="BR_joint">
+                <command_interface name="velocity">
+                    <param name="min">-10</param>
+                    <param name="max">10</param>
+                </command_interface>
+                <state_interface name="position"/>
+                <state_interface name="velocity"/>
+            </joint>
+        </ros2_control>
+    </xacro:unless>
+    <xacro:if value="$(arg sim_mode)">
+        <ros2_control name="GazeboSystem" type="system">
+            <hardware>
+                <plugin>gazebo_ros2_control/GazeboSystem</plugin>
+            </hardware>
+            <!-- <joint name="FL_joint">
                 <command_interface name="velocity">
                     <param name="min">-10</param>
@@ -28,44 +69,5 @@
                 <state_interface name="velocity"/>
                 <state_interface name="position"/>
-            </joint>
-            <joint name="BL_joint">
-                <command_interface name="velocity">
-                    <param name="min">-10</param>
-                    <param name="max">10</param>
-                </command_interface>
-                <state_interface name="velocity"/>
-                <state_interface name="position"/>
-            </joint>
-            <joint name="BR_joint">
-                <command_interface name="velocity">
-                    <param name="min">-10</param>
-                    <param name="max">10</param>
-                </command_interface>
-                <state_interface name="velocity"/>
-                <state_interface name="position"/>
-            </joint>
-        </ros2_control>
-    </xacro:unless>
-    <xacro:if value="$(arg sim_mode)">
-        <ros2_control name="GazeboSystem" type="system">
-            <hardware>
-                <plugin>gazebo_ros2_control/GazeboSystem</plugin>
-            </hardware>
-            <joint name="FL_joint">
-                <command_interface name="velocity">
-                    <param name="min">-10</param>
-                    <param name="max">10</param>
-                </command_interface>
-                <state_interface name="velocity"/>
-                <state_interface name="position"/>
-            </joint>
-            <joint name="FR_joint">
-                <command_interface name="velocity">
-                    <param name="min">-10</param>
-                    <param name="max">10</param>
-                </command_interface>
-                <state_interface name="velocity"/>
-                <state_interface name="position"/>
-            </joint>
+            </joint> -->
             <joint name="BL_joint">
                 <command_interface name="velocity">
