Commit message: made some modifications from knowledge of eyantra

File: cvr_bot_description/urdf/cvr_bot.xacro (robot description, xacro)
@@ -2,5 +2,5 @@
 <robot name="cvr_bot" xmlns:xacro="http://www.ros.org/wiki/xacro">
 <xacro:include filename="$(find cvr_bot_description)/urdf/materials.xacro" />
-<xacro:include filename="$(find cvr_bot_description)/urdf/cvr_bot.trans" />
+<!-- <xacro:include filename="$(find cvr_bot_description)/urdf/cvr_bot.trans" /> -->
 <xacro:include filename="$(find cvr_bot_description)/urdf/cvr_bot.gazebo" />
 <xacro:property name="base_mass" value="46.034" />

File: cvr_bot_description/urdf/cvr_bot_sim.xacro (robot description, xacro)
@@ -1,3 +1,3 @@
-<?xml version="1.0" ?>
+<?xml version="1.0"?>
 <robot name="cvr_bot" xmlns:xacro="http://www.ros.org/wiki/xacro">
 <xacro:include filename="$(find cvr_bot_description)/urdf/materials.xacro" />
@@ -6,5 +6,5 @@
 <xacro:property name="base_mass" value="2.034" />
 <xacro:property name="wheel_mass" value="0.8637" />
-<xacro:property name="wheel_radius" value="0.07"/>
+<xacro:property name="wheel_radius" value="0.0625"/>
 <xacro:macro name="box_inertia" params="b_mass b_x b_y b_z">
         <mass value="${b_mass}"/>
@@ -49,13 +49,13 @@
   </visual>
   <collision>
-    <origin xyz="0 0 0.115" rpy="0 0 0"/>
-    <geometry>
-      <!-- <mesh filename="package://cvr_bot_description/meshes/base_link.dae" scale="0.001 0.001 0.001"/> -->
-      <box size="0.29 0.29 0.23"/>
+    <origin xyz="0 0 0" rpy="0 0 0"/>
+    <geometry>
+      <mesh filename="file://$(find cvr_bot_description)/meshes/base_link.dae" scale="0.001 0.001 0.001"/>
+      <!-- <box size="0.29 0.29 0.23"/> -->
     </geometry>
   </collision>
 </link>
 <xacro:property name="wheel_inertia">
-    <xacro:cylinder_inertia c_mass="${wheel_mass}" r = "0.065" l="0.0471"/>   <!--  mass radius length of a wheel -->
+    <xacro:cylinder_inertia c_mass="${wheel_mass}" r = "0.0625" l="0.0471"/>   <!--  mass radius length of a wheel -->
 </xacro:property>
 <link name="br_wheel">
@@ -75,7 +75,9 @@
   <collision>
     <!-- <origin xyz="0.094914 0.152452 -0.064084" rpy="0 0 0"/> -->
-    <geometry>
-      <!-- <mesh filename="package://cvr_bot_description/meshes/br_wheel_2.dae" scale="0.001 0.001 0.001"/> -->
-      <sphere radius="${wheel_radius}"/>
+    <origin xyz="0.0 -0.015 0.0" rpy="1.57 0 0"/>
+    <geometry>
+      <!-- <mesh filename="file://$(find cvr_bot_description)/meshes/br_wheel_2.dae" scale="0.001 0.001 0.001"/> -->
+      <!-- <sphere radius="${wheel_radius}"/> -->
+      <cylinder length="0.045" radius="0.065"/>
     </geometry>
   </collision>
@@ -97,7 +99,9 @@
   <collision>
     <!-- <origin xyz="-0.095849 0.151214 -0.062584" rpy="0 0 0"/> -->
-    <geometry>
-      <!-- <mesh filename="package://cvr_bot_description/meshes/fr_wheel.dae" scale="0.001 0.001 0.001"/> -->
-      <sphere radius="${wheel_radius}"/>
+    <origin xyz="0.0 -0.015 0.0" rpy="1.57 0 0"/>
+    <geometry>
+      <!-- <mesh filename="file://$(find cvr_bot_description)/meshes/fr_wheel.dae" scale="0.001 0.001 0.001"/> -->
+      <!-- <sphere radius="${wheel_radius}"/> -->
+      <cylinder length="0.045" radius="0.065"/>
     </geometry>
   </collision>
@@ -119,7 +123,9 @@
   <collision>
     <!-- <origin xyz="-0.095849 -0.162786 -0.062584" rpy="0 0 0"/> -->
-    <geometry>
-      <!-- <mesh filename="package://cvr_bot_description/meshes/fl_wheel.dae" scale="0.001 0.001 0.001"/> -->
-      <sphere radius="${wheel_radius}"/>
+    <origin xyz="0.0 0.015 0.0" rpy="1.57 0 0"/>
+    <geometry>
+      <!-- <mesh filename="file://$(find cvr_bot_description)/meshes/fl_wheel.dae" scale="0.001 0.001 0.001"/> -->
+      <!-- <sphere radius="${wheel_radius}"/> -->
+      <cylinder length="0.045" radius="0.065"/>
     </geometry>
   </collision>
@@ -141,7 +147,9 @@
   <collision>
     <!-- <origin xyz="0.096151 -0.162786 -0.062584" rpy="0 0 0"/> -->
-    <geometry>
-      <!-- <mesh filename="package://cvr_bot_description/meshes/bl_wheel.dae" scale="0.001 0.001 0.001"/> -->
-      <sphere radius="${wheel_radius}"/>
+    <origin xyz="0.0 0.015 0.0" rpy="1.57 0 0"/>
+    <geometry>
+      <!-- <mesh filename="file://$(find cvr_bot_description)/meshes/bl_wheel.dae" scale="0.001 0.001 0.001"/> -->
+      <!-- <sphere radius="${wheel_radius}"/> -->
+      <cylinder length="0.045" radius="0.065"/>
     </geometry>
   </collision>

File: cvr_bot_description/urdf/robot.urdf.xacro (robot description, xacro)
@@ -4,10 +4,11 @@
     <xacro:arg name="sim_mode" default="false"/>
     <xacro:include filename="cvr_bot_sim.xacro" />
-    <xacro:if value="$(arg use_ros2_control)">
+    <xacro:include filename="ros2_control.xacro" />
+    <!-- <xacro:if value="$(arg use_ros2_control)">
         <xacro:include filename="ros2_control.xacro" />
     </xacro:if>
     <xacro:unless value="$(arg use_ros2_control)">
-        <xacro:include filename="gazebo_control.xacro" />
-    </xacro:unless>
+        <xacro:include filename="gazebo_control.gazebo" />
+    </xacro:unless> -->
     <!-- <xacro:include filename="lidar.xacro" />
     <xacro:include filename="camera.xacro" /> -->

File: cvr_bot_description/urdf/ros2_control.xacro (robot description, xacro)
@@ -88,9 +88,9 @@
         </ros2_control>
     </xacro:if>
-    <gazebo>
+    <!-- <gazebo>
         <plugin name="gazebo_ros2_control" filename="libgazebo_ros2_control.so">
             <parameters>$(find cvr_bot_description)/config/my_controllers.yaml</parameters>
             <parameters>$(find cvr_bot_description)/config/gaz_ros2_ctl_use_sim.yaml</parameters>
         </plugin>
-    </gazebo>
+    </gazebo> -->
 </robot>
