Commit message: changes made after testing on hardware

File: cvrbot_description/urdf/cvr_bot_sim.xacro (robot description, xacro)
@@ -4,5 +4,5 @@
   <xacro:arg name="is_sim" default="true"/>
 <xacro:include filename="$(find cvrbot_description)/urdf/materials.xacro" />
-<!-- <xacro:include filename="$(find cvrbot_description)/urdf/cvr_bot.trans" /> -->
+<xacro:include filename="$(find cvrbot_description)/urdf/cvr_bot.trans" />
 <xacro:include filename="$(find cvrbot_description)/urdf/cvr_gazebo.xacro" />
 <xacro:include filename="$(find cvrbot_description)/urdf/cvr_ros2_contol.xacro" />
@@ -210,5 +210,5 @@
     xyz="0 0 0" />
 </joint>
-<link name="laser">
+<link name="laser_link">
   <inertial>
     <origin xyz="-0.011945780406062 -0.000381929217680526 -0.0170649378129477" rpy="0 0 0" />
@@ -234,6 +234,7 @@
 <joint name="laser_joint" type="fixed">
   <origin xyz="0.080526 0.0 0.26" rpy="0 0 3.14" />
+  <!-- <origin xyz="-0.0050526 -0.0023221 0.1208" rpy="0 0 0" /> -->
   <parent link="cvr_bot_base_link" />
-  <child link="laser" />
+  <child link="laser_link" />
   <axis xyz="0 0 0" />
 </joint>

File: cvrbot_description/urdf/cvr_gazebo.xacro (robot description, xacro)
@@ -1,4 +1,4 @@
 <?xml version="1.0"?>
-<robot name="bumperbot" xmlns:xacro="http://ros.org/wiki/xacro">
+<robot name="cvr_bot" xmlns:xacro="http://ros.org/wiki/xacro">
 <xacro:property name="body_color" value="Gazebo/Black" />
   <!-- Move this one to ros2 control -->

File: cvrbot_description/urdf/cvr_ros2_contol.xacro (robot description, xacro)
@@ -1,4 +1,4 @@
 <?xml version="1.0"?>
-<robot xmlns:xacro="http://www.ros.org/wiki/xacro" name="bumperbot">
+<robot xmlns:xacro="http://www.ros.org/wiki/xacro" name="cvr_bot">
     <ros2_control name="RobotSystem" type="system">
         <!-- ros2_control Gazebo -->
@@ -11,14 +11,6 @@
         <xacro:unless value="$(arg is_sim)">
             <hardware>
-                <plugin>diffdrive_arduino/DiffDriveArduinoHardware</plugin>
-                <param name="left_wheel_name">BL_joint</param>
-                <param name="right_wheel_name">BR_joint</param>
-                <param name="left1_wheel_name">FL_joint</param>
-                <param name="right1_wheel_name">FR_joint</param>
-                <param name="loop_rate">30</param>
-                <param name="device">/dev/ttyUSB0</param>
-                <param name="baud_rate">57600</param>
-                <param name="timeout_ms">1000</param>
-                <param name="enc_counts_per_rev">2952</param>
+                <plugin>bumperbot_firmware/BumperbotInterface</plugin>
+                <param name="port">/dev/ttyACM0</param>
             </hardware>
         </xacro:unless>
@@ -46,5 +38,5 @@
         </joint>
         <!-- ros2_control Common Interfaces -->
-        <joint name="FR_joint">
+        <!-- <joint name="FR_joint">
             <command_interface name="velocity">
               <param name="min">-1</param>
@@ -61,5 +53,5 @@
             <state_interface name="position" />
             <state_interface name="velocity" />
-        </joint>
+        </joint> -->
     </ros2_control>
 </robot>
